File: pcb/kicad/xz1-direct.kicad_sch (KiCad schematic)
At the start: 7 parts, among them J1 PJ-327A0-SMT, J2 PJ-327A0-SMT

Commit message: pcb: Rev C-M2, jacks grouped next to the plug
Shorter lever on the plug when cables are plugged in: both jacks move
next to the plug, the wire pads move to the right, R1/R2 rotate and
the M2 holes move. Circuit, star ground and rules unchanged.

Co-Authored-By: Claude Opus 5.5 <noreply@anthropic.com>
Other:
- note added: "XZ1 STEREO SPLITTER / Rev C-M2"
- note removed: "XZ1 STEREO SPLITTER / Rev B"
